File: PCB/65MK/65MK.kicad_pcb (KiCad board)
At the start: 2 copper layers, 344.5 x 102.4 mm, 150 parts, among them SW1 RotaryEncoder_Switch

Commit message: 3d Models
Parts:
- moved D13 18.4 mm to (289.9, 110.3)
- moved D14 18.4 mm to (308.9, 110.3)
- moved D16 18.4 mm to (349.4, 110.3)
- moved D17 18.4 mm to (376.4, 112.7)
- moved D29 18.4 mm to (261.3, 129.4)
- moved D47 18.4 mm to (285.1, 148.4)
- moved D64 18.4 mm to (320.8, 167.5)
- moved D71 18.4 mm to (277.9, 186.5)
- moved D73 18.4 mm to (332.7, 191.3)
- moved MX14 18.4 mm to (305.7, 105.6)
- moved MX17 18.4 mm to (372.4, 105.6)
- moved MX29 18.4 mm to (277.2, 124.6)
- moved MX33 18.4 mm to (372.4, 124.6)
- moved MX46 18.4 mm to (281.9, 143.7)
- moved MX47 18.4 mm to (301.0, 143.7)
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
Commit message: Added Gerbers
Other:
- board size 344.5 x 102.4 mm -> 344.5 x 102.1 mm
Changed lines of the file:
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@@
     )
   )
-  (gr_arc (start 41.411186 197.64375) (mid 39.166122 196.713814) (end 38.236186 194.46875) (layer "Edge.Cuts") (width 0.1))
+  (gr_arc (start 119.38 191.008014) (mid 121.625068 191.937946) (end 122.555 194.183014) (layer "Edge.Cuts") (width 0.1))
+  (gr_arc (start 125.73 197.358014) (mid 123.484932 196.428082) (end 122.555 194.183014) (layer "Edge.Cuts") (width 0.1))
+  (gr_line (start 41.402 191.008014) (end 119.38 191.008014) (layer "Edge.Cuts") (width 0.1))
+  (gr_arc (start 41.402 191.008014) (mid 39.156927 190.078076) (end 38.227 187.833014) (layer "Edge.Cuts") (width 0.1))
   (gr_line (start 379.548686 95.25) (end 41.411186 95.25) (layer "Edge.Cuts") (width 0.1))
-  (gr_line (start 382.723686 194.46875) (end 382.723686 98.425) (layer "Edge.Cuts") (width 0.1))
+  (gr_line (start 382.723686 187.071) (end 382.723686 98.425) (layer "Edge.Cuts") (width 0.1))
+  (gr_arc (start 260.604 194.183056) (mid 261.533932 191.937988) (end 263.779 191.008056) (layer "Edge.Cuts") (width 0.1))
   (gr_arc (start 379.548686 95.25) (mid 381.793718 96.179954) (end 382.723686 98.425) (layer "Edge.Cuts") (width 0.1))
-  (gr_arc (start 382.723686 194.46875) (mid 381.793735 196.713799) (end 379.548686 197.64375) (layer "Edge.Cuts") (width 0.1))
-  (gr_line (start 41.411186 197.64375) (end 379.548686 197.64375) (layer "Edge.Cuts") (width 0.1))
-  (gr_line (start 38.236186 98.425) (end 38.236186 194.46875) (layer "Edge.Cuts") (width 0.1))
+  (gr_arc (start 382.723686 187.071) (mid 381.793724 189.316014) (end 379.548686 190.246) (layer "Edge.Cuts") (width 0.1))
+  (gr_arc (start 260.604 194.183) (mid 259.674068 196.428068) (end 257.429 197.358) (layer "Edge.Cuts") (width 0.1))
+  (gr_arc (start 376.373686 193.421) (mid 375.44375 195.666064) (end 373.198686 196.596) (layer "Edge.Cuts") (width 0.1))
+  (gr_line (start 323.977 196.596) (end 373.198686 196.596) (layer "Edge.Cuts") (width 0.1))
+  (gr_line (start 263.779 191.008056) (end 317.627 191.008) (layer "Edge.Cuts") (width 0.1))
+  (gr_arc (start 323.977 196.596) (mid 321.897861 195.75768) (end 320.802 193.802) (layer "Edge.Cuts") (width 0.1))
+  (gr_line (start 125.73 197.358014) (end 257.429 197.358) (layer "Edge.Cuts") (width 0.1))
+  (gr_line (start 38.236186 98.425) (end 38.227 187.833014) (layer "Edge.Cuts") (width 0.1))
+  (gr_arc (start 317.627 191.008) (mid 319.708042 191.844156) (end 320.802 193.802) (layer "Edge.Cuts") (width 0.1))
   (gr_arc (start 38.236186 98.425) (mid 39.166122 96.179936) (end 41.411186 95.25) (layer "Edge.Cuts") (width 0.1))
+  (gr_arc (start 376.373686 193.421056) (mid 377.303594 191.175964) (end 379.548686 190.246056) (layer "Edge.Cuts") (width 0.1))
   (segment (start 49.507436 103.02875) (end 47.207936 100.72925) (width 0.25) (layer "F.Cu") (net 1))
   (segment (start 47.207936 100.72925) (end 45.697436 100.72925) (width 0.25) (layer "F.Cu") (net 1))
@@
   (via (at 50.936186 184.15) (size 0.8) (drill 0.4) (layers "F.Cu" "B.Cu") (net 96))
   (segment (start 189.692436 188.18125) (end 111.261186 188.18125) (width 0.25) (layer "B.Cu") (net 96))
+  (segment (start 319.88025 188.18125) (end 324.64275 192.94375) (width 0.25) (layer "B.Cu") (net 96))
+  (segment (start 324.64275 192.94375) (end 332.717436 192.94375) (width 0.25) (layer "B.Cu") (net 96))
   (segment (start 351.767436 192.94375) (end 370.817436 192.94375) (width 0.25) (layer "B.Cu") (net 96))
   (segment (start 194.604936 192.94375) (end 194.454936 192.94375) (width 0.25) (layer "B.Cu") (net 96))
-  (segment (start 308.904936 192.94375) (end 332.717436 192.94375) (width 0.25) (layer "B.Cu") (net 96))
   (segment (start 194.454936 192.94375) (end 189.692436 188.18125) (width 0.25) (layer "B.Cu") (net 96))
   (segment (start 194.604936 192.94375) (end 199.367436 188.18125) (width 0.25) (layer "B.Cu") (net 96))
@@
   (segment (start 332.717436 192.94375) (end 351.767436 192.94375) (width 0.25) (layer "B.Cu") (net 96))
   (segment (start 277.948686 188.18125) (end 304.142436 188.18125) (width 0.25) (layer "B.Cu") (net 96))
-  (segment (start 304.142436 188.18125) (end 308.904936 192.94375) (width 0.25) (layer "B.Cu") (net 96))
   (segment (start 50.936186 184.15) (end 54.967436 188.18125) (width 0.25) (layer "B.Cu") (net 96))
+  (segment (start 304.142436 188.18125) (end 319.88025 188.18125) (width 0.25) (layer "B.Cu") (net 96))
   (segment (start 54.967436 188.18125) (end 56.492436 188.18125) (width 0.25) (layer "B.Cu") (net 96))
   (segment (start 56.492436 188.18125) (end 85.067436 188.18125) (width 0.25) (layer "B.Cu") (net 96))
